Commit message: Add RViz arm overlays

File: dvrk_model/model/PSM1.urdf.xacro (robot description, xacro)
@@ -3,8 +3,8 @@
   <!-- Macros -->
   <xacro:include filename="$(find dvrk_model)/model/psm.urdf.xacro"/>
-  <link name="world"/>
+  <link name="PSM1_base"/>
   <xacro:psm_sca
       prefix="PSM1_"
-      parent_link="world"
-      xyz="-0.25 0.0 0.5" rpy="0.0 0.0 3.1415926"/>
+      parent_link="PSM1_base"
+      xyz="0.0 0.0 0.0" rpy="0.0 0.0 0.0"/>
 </robot>

File: dvrk_model/model/PSM2.urdf.xacro (robot description, xacro)
@@ -3,8 +3,8 @@
   <!-- Macros -->
   <xacro:include filename="$(find dvrk_model)/model/psm.urdf.xacro"/>
-  <link name="world"/>
+  <link name="PSM2_base"/>
   <xacro:psm_caudier
       prefix="PSM2_"
-      parent_link="world"
-      xyz="0.25 0.0 0.5" rpy="0.0 0.0 -3.1415926"/>
+      parent_link="PSM2_base"
+      xyz="0.0 0.0 0.0" rpy="0.0 0.0 0.0"/>
 </robot>

File: dvrk_model/model/PSM3.urdf.xacro (robot description, xacro)
@@ -3,8 +3,8 @@
   <!-- Macros -->
   <xacro:include filename="$(find dvrk_model)/model/psm.urdf.xacro"/>
-  <link name="world"/>
+  <link name="PSM3_base"/>
   <xacro:psm_caudier
     prefix="$(arg prefix)"
-    parent_link="world"
-    xyz="0.50 0.0 0.5" rpy="0.0 0.0 -3.1415926"/>
+    parent_link="PSM3_base"
+    xyz="0.0 0.0 0.0" rpy="0.0 0.0 0.0"/>
 </robot>
